File: hardware/cipinkoklingacik.kicad_sch (KiCad schematic)
At the start: 92 parts, among them J1 GLITCH/GND, J2 TARGET/GND, J3 RESET/GND, J4 TRIGGER/GND, J5 UART, Q1 AO3400A, Q2 Si2377EDS, Q3 Si2377EDS, Q4 2N7002, Q5 2N7002, Q6 2N7002, U1 Raspberry Pi Pico 2, U2 UCC27517DBVR, U3 NX3L1T3157GMZ, U4 AP2112K-3.3, U5 AP2112K-1.8, U6 TLV70436DBVR, U7 SN74LVC1G17, U8 SN74AXC4T774PWR

Commit message: Prepare C4 alpha.2 with stocked sourcing and DFM audit fixes
Parts:
- C1: LCSC (none) -> C97954
- C10, C11, C14, C3, C5, C6, C8: LCSC (none) -> C77079
- C12, C13, C16, C17, C18, C2: LCSC (none) -> C49678; MPN GRM21BR71H104KA01L -> CC0805KRX7R9BB104; Manufacturer Murata -> Yageo
- C4, C7, C9: LCSC (none) -> C128532
- D1: LCSC (none) -> C124205
- D2: LCSC (none) -> C98221
- F1: LCSC (none) -> C99561; MPN MF-NSMF025X-2 -> 1206L025YR; Manufacturer Bourns -> Littelfuse; Requirement 250 mA hold, 16 V PTC; drop/trip curve require review, NOT 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 -> 250 mA hold, 500 mA trip, 16 V PTC; 100 A fault rating; R1m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
- Q1: LCSC (none) -> C20917
- Q2, Q3: LCSC (none) -> C143698
- Q4, Q5, Q6: LCSC (none) -> C65189
- R1, R10, R17, R19, R2, R21, R23, R24, R26, R28, R3, R30, R31, R34, R37, R4, R5, R6, R9: LCSC (none) -> C17414; MPN RC0805FR-0710KL -> 0805W8F1002T5E; Manufacturer Yageo -> UNI-ROYAL
- R11, R12: LCSC (none) -> C17630; MPN RC0805FR-07330RL -> 0805W8F3300T5E; Manufacturer Yageo -> UNI-ROYAL
- R13, R32, R35, R7, R8: LCSC (none) -> C17513; MPN RC0805FR-071KL -> 0805W8F1001T5E; Manufacturer Yageo -> UNI-ROYAL
- R14, R33: LCSC (none) -> C149504; MPN RC0805FR-07100KL -> 0805W8F1003T5E; Manufacturer Yageo -> UNI-ROYAL
- R15, R16: value 15 1% >=1W -> 15 1% 2W; LCSC (none) -> C6639259; MPN CRCW251215R0FKEGHP -> RC2512FK-7W15RL; Manufacturer Vishay -> Yageo; Requirement 15 ohm 1%, high-pulse series; qualify >=1 W on actual PCB a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 -> 15 ohm 1%, 2 W (7W power code); <=0.756 W bounded peak, no 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
- R18, R22, R25, R29, R36, R38: LCSC (none) -> C17408; MPN RC0805FR-07100RL -> 0805W8F1000T5E; Manufacturer Yageo -> UNI-ROYAL
- R27: LCSC (none) -> C17521; MPN RC0805FR-072R2L -> 0805W8F220KT5E; Manufacturer Yageo -> UNI-ROYAL
- R39: LCSC (none) -> C17888; MPN RC1206JR-070RL -> 1206W4F0000T5E; Manufacturer Yageo -> UNI-ROYAL
- U2: LCSC (none) -> C99395
- U3: LCSC (none) -> C1870392
- U4: LCSC (none) -> C51118
- U5: LCSC (none) -> C176944
- U6: value TLV70436DBVR -> TPS7A2036PDBVR; LCSC (none) -> C2873626; MPN TLV70436DBVR -> TPS7A2036PDBVR; Requirement 3.6 V; pinout differs from AP2112 -> 3.6 V; IN1 GND2 EN3 NC4 OUT5; EN tied to HOLD_IN, not Pico/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
- U7: LCSC (none) -> C7836
Connections:
- net GND: now also U6.2 (GND); no longer U6.1 (GND)
- net HOLD: now also U6.1 (IN), U6.3 (EN); no longer U6.2 (IN)
- net MVCC: now also U6.5 (OUT); no longer U6.3 (OUT)
- no-connect marks 26 -> 25
Other:
- note added: "C4 ENGINEERING PROTOTYPE - HARDWARE UNQUALIFIED"
- note removed: "C3 ENGINEERING PROTOTYPE - HARDWARE UNQUALIFIED"
- title: ČipinkoKlingáčik C3 - engineering prototype -> ČipinkoKlingáčik C4 - engineering prototype
